File: InspireFly-Ardunio-Workshop.kicad_sch (KiCad schematic)
At the start: 25 parts, among them J1 10118194-0001LF, J2 Conn_01x13, J3 Conn_01x18, U1 ATMEGA328-PU, U2 FT231XS-U, U3 IC REG LINEAR 3.3V, Y1 Crystal

Commit message: First Push
Parts:
- removed C1, C2: 22pF, Capacitor_SMD:C_0603_1608Metric_Pad1.08x0.95mm_HandSolder, symbol Device:C
- removed C10, C12, C3, C4, C5, C9: 100nF, Capacitor_SMD:C_0603_1608Metric_Pad1.08x0.95mm_HandSolder, symbol Device:C
- removed C11: 10nF, Capacitor_SMD:C_0603_1608Metric_Pad1.08x0.95mm_HandSolder, symbol Device:C
- removed C13: 10uF, Capacitor_SMD:C_1206_3216Metric_Pad1.33x1.80mm_HandSolder, symbol Device:C
- removed C14: 4.7uF, Capacitor_SMD:C_1206_3216Metric_Pad1.33x1.80mm_HandSolder, symbol Device:C
- removed C7, C8: 47pF, Capacitor_SMD:C_0603_1608Metric_Pad1.08x0.95mm_HandSolder, symbol Device:C
- removed FB1: FerriteBead, Inductor_SMD:L_0603_1608Metric_Pad1.05x0.95mm_HandSolder, symbol Device:FerriteBead
- removed J1: 10118194-0001LF, InspireFly_ARD-Workshop-FtpLib:AMPHENOL_10118194-0001LF, symbol InspireFly_ARD-Workshop-Symlib:10118194-0001LF
- removed JP1: SolderJumper_3_Open, Jumper:SolderJumper-3_P1.3mm_Open_RoundedPad1.0x1.5mm_NumberLabels, symbol Jumper:SolderJumper_3_Open
- removed R1: 10K, Resistor_SMD:R_0603_1608Metric_Pad0.98x0.95mm_HandSolder, symbol Device:R_US
- removed R2, R3: 27, Resistor_SMD:R_0603_1608Metric_Pad0.98x0.95mm_HandSolder, symbol Device:R_US
- removed U1: ATMEGA328-PU, InspireFly_ARD-Workshop-FtpLib:DIP787W46P254L3467H508Q28, symbol InspireFly_ARD-Workshop-Symlib:ATMEGA328-PU
- removed U2: FT231XS-U, InspireFly_ARD-Workshop-FtpLib:FT231XS-U, symbol InspireFly_ARD-Workshop-Symlib:FT231XS-U
- removed U3: IC REG LINEAR 3.3V, InspireFly_ARD-Workshop-FtpLib:SOT-223_DIO, symbol InspireFly_ARD-Workshop-Symlib:IC REG LINEAR 3.3V
- removed Y1: Crystal, InspireFly_ARD-Workshop-FtpLib:XTAL_ECS-160-20-46X, symbol Device:Crystal
Connections:
- net A4: no longer J3.2 (Pin_2)
- net A5: no longer J3.1 (Pin_1)
- new net SCL: J3.1 (Pin_1)
- new net SDA: J3.2 (Pin_2)
- no-connect marks 10 -> 0
